File: CurcuitV1/CurcuitV1.kicad_pcb (KiCad board)
At the start: 2 copper layers, 44 parts, among them J1 Conn_01x07, J2 Conn_01x03, J3 Conn_01x02, Q1 Q_NMOS_DGS, Q2 Q_NMOS_DGS, Q3 Q_NMOS_DGS, Q4 Q_NMOS_DGS, Q5 Q_NMOS_DGS, Q6 Q_NMOS_DGS, SW1 SW_Push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

Commit message: 基板外径仮案
Parts:
- added IC1: AS5600-ASOT, Package_SO:SOIC-8_3.9x4.9mm_P1.27mm, B.Cu at (120.0, 120.0)
- added J4: Conn_01x02, Connector_JST:JST_XH_S2B-XH-A_1x02_P2.50mm_Horizontal, F.Cu at (130.5, 112.2)
- moved R3 49.8 mm to (122.5, 116.2)
- moved C1 49.8 mm to (113.0, 120.5)
- moved C2 49.8 mm to (111.0, 115.5)
- moved C3 49.8 mm to (111.0, 124.2)
- moved C4 49.8 mm to (113.0, 129.2)
- moved C5 49.8 mm to (111.0, 133.0)
- moved C6 49.8 mm to (113.0, 138.0)
- moved D1 49.8 mm to (113.0, 116.2)
- moved D2 49.8 mm to (113.0, 125.0)
- moved D3 49.8 mm to (113.0, 133.8)
- moved Q1 49.8 mm to (125.5, 120.0)
- moved Q2 49.8 mm to (125.5, 116.0)
- moved Q3 49.8 mm to (125.5, 128.8)
- moved Q4 49.8 mm to (125.5, 124.8)
- moved Q5 49.8 mm to (125.5, 137.5)
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Connections:
- SW1 pad 1: unconnected-(SW1-Pad1) -> GND
- SW1 pad 2: unconnected-(SW1-Pad2) -> NSRT
- U4 pad 2: unconnected-(U4-PF0-Pad2) -> Net-(U4-PF0)
- U4 pad 3: unconnected-(U4-PF1-Pad3) -> Net-(U4-PF1)
- Y2 pad 1: unconnected-(Y2-Pad1) -> Net-(U4-PF0)
- Y2 pad 2: unconnected-(Y2-Pad2) -> GND
- Y2 pad 3: unconnected-(Y2-Pad3) -> Net-(U4-PF1)
Other:
- board outline added: 40 x 40 mm

Commit message: 大体完成
Parts:
- added C12: 10u, Capacitor_SMD:C_0805_2012Metric, F.Cu at (132.5, 134.2)
- added C13: 10u, Capacitor_SMD:C_0805_2012Metric, F.Cu at (132.5, 137.2)
- added C14: 10u, Capacitor_SMD:C_0805_2012Metric, F.Cu at (111.0, 112.5)
- added C15: 10u, Capacitor_SMD:C_0805_2012Metric, F.Cu at (109.0, 112.5)
- added C16: 10u, Capacitor_SMD:C_0805_2012Metric, F.Cu at (107.0, 112.5)
- added D5: D_Schottky, Diode_SMD:D_SOD-323_HandSoldering, F.Cu at (128.8, 138.0)
- added D6: LED, LED_SMD:LED_0603_1608Metric, F.Cu at (101.8, 109.2)
- added D7: LED, LED_SMD:LED_0603_1608Metric, F.Cu at (101.8, 107.2)
- added D8: LED, LED_SMD:LED_0603_1608Metric, F.Cu at (107.2, 101.8)
- added D9: LED, LED_SMD:LED_0603_1608Metric, F.Cu at (109.2, 101.8)
- added H1: MountingHole, MountingHole:MountingHole_3.2mm_M3_DIN965_Pad, F.Cu at (137.0, 103.0)
- added H2: MountingHole, MountingHole:MountingHole_3.2mm_M3_DIN965_Pad, F.Cu at (103.0, 103.0)
- added H3: MountingHole, MountingHole:MountingHole_3.2mm_M3_DIN965_Pad, F.Cu at (103.0, 137.0)
- added H4: MountingHole, MountingHole:MountingHole_3.2mm_M3_DIN965_Pad, F.Cu at (137.0, 137.0)
- added R14: 10k, Resistor_SMD:R_0603_1608Metric, F.Cu at (123.5, 103.8)
- added R15: 1k, Resistor_SMD:R_0603_1608Metric, F.Cu at (104.8, 109.2)
- added R16: 1k, Resistor_SMD:R_0603_1608Metric, F.Cu at (104.8, 107.2)
- added R17: 1k, Resistor_SMD:R_0603_1608Metric, F.Cu at (107.2, 104.8)
- added R18: 1k, Resistor_SMD:R_0603_1608Metric, F.Cu at (109.2, 104.8)
- added SW2: SW_Push, Button_Switch_SMD:SW_Push_1P1T_NO_Vertical_Wuerth_434133025816, F.Cu at (126.5, 103.5)
- added U6: AP7375-3.3, Package_TO_SOT_SMD:SOT-23, F.Cu at (128.8, 135.0)
- U5: value LM1117MP-3.3 -> AP7375-3.3; footprint Package_TO_SOT_SMD:SOT-223-3_TabPin2 -> Package_TO_SOT_SMD:SOT-23
- moved J1 15.2 mm to (101.5, 127.6), turned to 180 degrees
- moved C7 10.8 mm to (120.8, 113.0), turned to -90 degrees
- moved U5 6.60 mm to (125.8, 113.0), turned to -90 degrees
- moved C8 5.53 mm to (125.8, 110.0)
- moved R13 4.53 mm to (111.2, 109.0)
- moved C10 4.51 mm to (122.8, 101.5)
- moved C9 4.51 mm to (113.0, 111.2)
- moved U4 4.51 mm to (117.5, 106.0)
- moved Y2 4.51 mm to (116.0, 112.5)
- moved C11 3.58 mm to (118.8, 112.8), turned to 90 degrees
- moved C1 2.85 mm to (110.2, 121.2), turned to 0 degrees
- moved C4 2.76 mm to (110.2, 129.5), turned to 0 degrees
- moved C6 2.76 mm to (110.2, 137.8), turned to 0 degrees
- moved C2 2.36 mm to (109.0, 116.8)
- moved D1 2.36 mm to (111.0, 117.5)
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Connections:
- J1 pad 3: unconnected-(J1-Pin_3-Pad3) -> NSRT
- J1 pad 4: unconnected-(J1-Pin_4-Pad4) -> SWDIO
- J1 pad 5: unconnected-(J1-Pin_5-Pad5) -> SWCLK
- J1 pad 6: unconnected-(J1-Pin_6-Pad6) -> PC_TX
- J1 pad 7: unconnected-(J1-Pin_7-Pad7) -> PC_RX
- J4 pad 1: GND -> UART2_TX
- J4 pad 2: VCC -> UART2_RX
- U4 pad 12: unconnected-(U4-PA6-Pad12) -> U_IN
- U4 pad 13: unconnected-(U4-PA7-Pad13) -> V_IN
- U4 pad 14: unconnected-(U4-PB0-Pad14) -> W_IN
- U4 pad 15: unconnected-(U4-PB1-Pad15) -> BUTTON
- U4 pad 29: unconnected-(U4-PB6-Pad29) -> PC_TX
- U4 pad 30: unconnected-(U4-PB7-Pad30) -> PC_RX
- U4 pad 8: unconnected-(U4-PA2-Pad8) -> UART2_TX
- U4 pad 9: unconnected-(U4-PA3-Pad9) -> UART2_RX
Routing:
- net +3V3: track 0.00 -> 67.3 mm, vias 0 -> 2
- net W_IN: track 0.00 -> 48.4 mm, vias 0 -> 2
- net +5V: track 25.2 -> 71.5 mm, vias 0 -> 4
- net NSRT: track 0.00 -> 40.8 mm, vias 0 -> 2
- net V_IN: track 0.00 -> 38.9 mm, vias 0 -> 2
- net VCC: track 24.6 -> 63.2 mm, vias 0 -> 11
- net SWDIO: track 0.00 -> 24.0 mm, vias 0 -> 1
- net SWCLK: track 0.00 -> 21.1 mm, vias 0 -> 1
- net PC_TX: track 0.00 -> 15.4 mm
- net U_IN: track 0.00 -> 15.3 mm, vias 0 -> 2
- net PC_RX: track 0.00 -> 14.0 mm, vias 0 -> 1
- net UART2_TX: track 0.00 -> 12.5 mm
- net V_OUT: track 4.61 -> 15.4 mm
- net W_OUT: track 4.61 -> 14.8 mm
- net UART2_RX: track 0.00 -> 9.88 mm
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- added copper zone on B.Cu, net GND
- added copper zone on F.Cu, net GND
- added copper zone on F.Cu, net U_OUT
- added copper zone on B.Cu, net VCC
- added copper zone on F.Cu, net VCC
- added copper zone on F.Cu, net V_OUT
- added copper zone on F.Cu, net W_OUT
Other:
- outline, holes or cut-outs redrawn
- board text added: "+"
- board text added: "-"
- board text added: "3V3"
- board text added: "BLDC Driver V1.0 Designed by Bambi"
- board text added: "CLK"
- board text added: "DIO"
- board text added: "GND"
- board text added: "NSRT"
- board text added: "RX"
- board text added: "TX"
- board text added: "U"
- board text added: "V"
- board text added: "W"

Commit message: LED配線
Connections:
- U4 pad 25: unconnected-(U4-PA15-Pad25) -> LED1
- U4 pad 26: unconnected-(U4-PB3-Pad26) -> LED2
- U4 pad 27: unconnected-(U4-PB4-Pad27) -> LED3
- U4 pad 28: unconnected-(U4-PB5-Pad28) -> LED4
Routing:
- net LED1: track 0.00 -> 13.0 mm, vias 0 -> 2
- net LED2: track 0.00 -> 9.29 mm, vias 0 -> 2
- net LED3: track 0.00 -> 6.40 mm
- net LED4: track 0.00 -> 4.09 mm

Commit message: 発注した
Parts:
- added C17: 10u, Capacitor_SMD:C_0805_2012Metric, F.Cu at (105.0, 124.5)
- added C18: 10u, Capacitor_SMD:C_0805_2012Metric, F.Cu at (105.0, 126.5)
- added C19: 10u, Capacitor_SMD:C_0805_2012Metric, F.Cu at (105.0, 128.5)
- added C20: 10u, Capacitor_SMD:C_0805_2012Metric, F.Cu at (105.0, 130.5)
- added C21: 10u, Capacitor_SMD:C_0805_2012Metric, F.Cu at (105.0, 132.5)
- added C22: 10u, Capacitor_SMD:C_0805_2012Metric, F.Cu at (105.0, 122.5)
- added C23: 10u, Capacitor_SMD:C_0805_2012Metric, F.Cu at (105.0, 120.5)
- added C24: 10u, Capacitor_SMD:C_0805_2012Metric, F.Cu at (105.0, 118.5)
- added C25: 10u, Capacitor_SMD:C_0805_2012Metric, F.Cu at (105.0, 116.5)
- added C26: 0.1u, Capacitor_SMD:C_0603_1608Metric, F.Cu at (102.5, 131.0)
- added D10: LED, LED_SMD:LED_0603_1608Metric, F.Cu at (108.2, 109.2)
- added R19: 1k, Resistor_SMD:R_0603_1608Metric, F.Cu at (104.8, 112.5)
- moved IC1 1.00 mm to (120.0, 120.0)
Connections:
- C1 pad 1: Net-(D1-K) -> VCC
- C4 pad 1: Net-(D2-K) -> VCC
- C6 pad 1: Net-(D3-K) -> VCC
- D1 pad 1: Net-(D1-K) -> VCC
- D2 pad 1: Net-(D2-K) -> VCC
- D3 pad 1: Net-(D3-K) -> VCC
- U4 pad 11: unconnected-(U4-PA5-Pad11) -> ENCODER_OUT
Routing:
- net VCC: track 63.2 -> 127.7 mm, vias 11 -> 14
- net GND: track 2.72 -> 31.2 mm, vias 3 -> 72
- net ENCODER_OUT: track 0.00 -> 12.3 mm, vias 0 -> 1
- net +3V3: track 67.3 -> 73.1 mm, vias 2 -> 3
- net Net-(D10-A): track 0.00 -> 3.72 mm
- net Net-(D3-K): track 2.80 -> 0.00 mm
- net Net-(D2-K): track 2.80 -> 0.00 mm
- net Net-(D1-K): track 2.80 -> 0.00 mm
- net U_IN: track 15.3 -> 12.7 mm
- net V_OUT: track 15.4 -> 13.5 mm
- net W_OUT: track 14.8 -> 12.8 mm
- net +5V: track 71.5 -> 70.6 mm, vias 4 -> 6
- net PC_TX: vias 0 -> 1
Other:
- board text added: "F303K8"

Commit message: V1.1発注
Parts:
- removed U6: AP7375-3.3, Package_TO_SOT_SMD:SOT-23
- added TP1: TestPoint, TestPoint:TestPoint_Pad_D2.0mm, B.Cu at (137.0, 123.2)
- added TP2: TestPoint, TestPoint:TestPoint_Pad_D2.0mm, B.Cu at (137.0, 120.0)
- added TP3: TestPoint, TestPoint:TestPoint_Pad_D2.0mm, B.Cu at (137.0, 116.8)
- added U7: AP7375-3.3, Package_TO_SOT_SMD:SOT-23, F.Cu at (125.8, 113.0)
- U5: value AP7375-3.3 -> AP7375-5
- moved U5 22.3 mm to (129.2, 135.0), turned to 90 degrees
- moved C12 0.35 mm to (132.8, 134.0)
- moved C13 0.25 mm to (132.2, 137.2)
- moved D5 0.25 mm to (129.0, 138.0)
Connections:
- J1 pad 3: NSRT -> SWDIO
- J1 pad 4: SWDIO -> SWCLK
- J1 pad 5: SWCLK -> NSRT
- U5 pad 1: GND -> VCC
- U5 pad 2: +3V3 -> +5V
- U5 pad 3: VCC -> GND
Routing:
- net U_OUT: track 12.8 -> 19.6 mm
- net W_OUT: track 12.8 -> 19.7 mm
- net V_OUT: track 13.5 -> 20.0 mm
- net NSRT: track 40.8 -> 43.7 mm, vias 2 -> 3
- net SWDIO: track 24.0 -> 26.5 mm
- net SWCLK: track 21.1 -> 23.6 mm
- net GND: track 31.2 -> 33.6 mm, vias 72 -> 89
- net VCC: track 127.7 -> 130.0 mm, vias 14 -> 15
- net +5V: track 70.6 -> 69.2 mm
- net Net-(Q5-G): track 7.31 -> 6.52 mm
- net Net-(Q3-G): track 7.31 -> 6.56 mm
Other:
- board text added: "BLDC Driver V1.1 Designed by Bambi"
- board text removed: "BLDC Driver V1.0 Designed by Bambi"
- board text removed: "F303K8"
