File: CurcuitV1/CurcuitV1.kicad_sch (KiCad schematic)
At the start: 38 parts, among them J1 Conn_01x07, Q1 Q_NMOS_DGS, Q2 Q_NMOS_DGS, Q3 Q_NMOS_DGS, Q4 Q_NMOS_DGS, Q5 Q_NMOS_DGS, Q6 Q_NMOS_DGS, SW1 SW_Push, U1 IR2302, U2 IR2302, U3 IR2302, U4 STM32F303K8Tx, U5 LM1117MP-3.3

Commit message: 水晶追加など
Parts:
- added C10, C11, C9: 0.1u, Capacitor_SMD:C_0603_1608Metric, symbol Device:C
- added J2: Conn_01x03, Connector_JST:JST_XH_S3B-XH-A_1x03_P2.50mm_Horizontal, symbol Connector_Generic:Conn_01x03
- added J3: Conn_01x02, Connector_JST:JST_XH_S2B-XH-A_1x02_P2.50mm_Horizontal, symbol Connector_Generic:Conn_01x02
- added Y2: CSTNE16M0V530000R0, CSTNE16M0V530000R0:OSC_CSTNE16M0V530000R0, symbol CSTNE16M0V530000R0:CSTNE16M0V530000R0
- D4: footprint (none) -> Diode_SMD:D_SOD-323_HandSoldering
Connections:
- net +3V3: now also C10.2, C11.2, C9.2
- net GND: now also C10.1, C11.1, C9.1, J3.1 (Pin_1)
- net U_OUT: now also J2.3 (Pin_3)
- net VCC: now also J3.2 (Pin_2)
- net V_OUT: now also J2.2 (Pin_2)
- net W_OUT: now also J2.1 (Pin_1)
- net NSRT: now reaches U4.4 (NRST)

Commit message: 基板外径仮案
Parts:
- added IC1: AS5600-ASOT, Package_SO:SOIC-8_3.9x4.9mm_P1.27mm, symbol AS5600-ASOT:AS5600-ASOT
- added J4: Conn_01x02, Connector_JST:JST_XH_S2B-XH-A_1x02_P2.50mm_Horizontal, symbol Connector_Generic:Conn_01x02
Connections:
- net +3V3: now also IC1.1 (VDD5V), IC1.2 (VDD3V3)
- net GND: now also SW1.1, Y2.2, IC1.4 (GND), J4.1 (Pin_1)
- net NSRT: now also SW1.2
- net VCC: now also J4.2 (Pin_2)
- net at Y2.1: now also U4.2 (PF0)
- net at Y2.3: now also U4.3 (PF1)
- new net ENCODER_OUT: IC1.3 (OUT)
Other:
- moved on the sheet: SW1

Commit message: 大体完成
Parts:
- added C12, C13, C14, C15, C16: 10u, Capacitor_SMD:C_0805_2012Metric, symbol Device:C
- added D5: D_Schottky, Diode_SMD:D_SOD-323_HandSoldering, symbol Device:D_Schottky
- added D6, D7, D8, D9: LED, LED_SMD:LED_0603_1608Metric, symbol Device:LED
- added H1, H2, H3, H4: MountingHole, MountingHole:MountingHole_3.2mm_M3_DIN965_Pad, symbol Mechanical:MountingHole
- added R14: 10k, Resistor_SMD:R_0603_1608Metric, symbol Device:R
- added R15, R16, R17, R18: 1k, Resistor_SMD:R_0603_1608Metric, symbol Device:R
- added SW2: SW_Push, Button_Switch_SMD:SW_Push_1P1T_NO_Vertical_Wuerth_434133025816, symbol Switch:SW_Push
- added U6: AP7375-3.3, Package_TO_SOT_SMD:SOT-23, symbol Regulator_Linear:LM1117MP-3.3
- U5: value LM1117MP-3.3 -> AP7375-3.3; footprint Package_TO_SOT_SMD:SOT-223-3_TabPin2 -> Package_TO_SOT_SMD:SOT-23
Connections:
- net +3V3: now also SW2.2
- net +5V: now also C13.1, D5.2 (A), U6.2 (VO)
- net GND: now also C12.2, C13.2, C14.1, C15.1, C16.1, D6.1 (K), D7.1 (K), D8.1 (K), D9.1 (K), R14.2, U6.1 (GND); no longer J4.1 (Pin_1)
- net NSRT: now also J1.3 (Pin_3)
- net SWCLK: now also J1.5 (Pin_5)
- net SWDIO: now also J1.4 (Pin_4)
- net U_IN: now also U4.12 (PA6)
- net VCC: now also C12.1, C14.2, C15.2, C16.2, D5.1 (K), U6.3 (VI); no longer J4.2 (Pin_2)
- net V_IN: now also U4.13 (PA7)
- net W_IN: now also U4.14 (PB0)
- net BUTTON: now reaches U4.15 (PB1)
- net BUTTON: now also R14.1, SW2.1
- net PC_TX: now reaches U4.29 (PB6)
- net PC_TX: now also J1.6 (Pin_6)
- net PC_RX: now reaches U4.30 (PB7)
- net PC_RX: now also J1.7 (Pin_7)
- net UART2_TX: now reaches U4.8 (PA2)
- net UART2_TX: now also J4.1 (Pin_1)
- net UART2_RX: now reaches U4.9 (PA3)
- net UART2_RX: now also J4.2 (Pin_2)
- new net: D7.2 (A), R16.1
- new net: D8.2 (A), R17.1
- new net: D6.2 (A), R15.1
- new net: D9.2 (A), R18.1
- new net LED1: R15.2
- new net LED2: R16.2
- new net LED3: R17.2
- new net LED4: R18.2

Commit message: LED配線
Connections:
- net LED1: now also U4.25 (PA15)
- net LED2: now also U4.26 (PB3)
- net LED3: now also U4.27 (PB4)
- net LED4: now also U4.28 (PB5)
Changed lines of the file:
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@@
+	(wire
+		(pts
+			(xy 86.36 76.2) (xy 88.9 76.2)
+		)
+		(stroke
+			(width 0)
+			(type default)
+		)
+	)
 	(wire
 		(pts
@@
 	(wire
 		(pts
+			(xy 55.88 63.5) (xy 58.42 63.5)
+		)
+		(stroke
+			(width 0)
+			(type default)
+		)
+	)
+	(wire
+		(pts
 			(xy 86.36 55.88) (xy 88.9 55.88)
 		)
@@
 	(wire
 		(pts
+			(xy 55.88 60.96) (xy 58.42 60.96)
+		)
+		(stroke
+			(width 0)
+			(type default)
+		)
+	)
+	(wire
+		(pts
 			(xy 86.36 73.66) (xy 88.9 73.66)
 		)
@@
 	(wire
 		(pts
+			(xy 55.88 66.04) (xy 58.42 66.04)
+		)
+		(stroke
+			(width 0)
+			(type default)
+		)
+	)
+	(wire
+		(pts
 			(xy 55.88 68.58) (xy 58.42 68.58)
 		)
@@
 		)
 	)
+	(global_label "LED2"
+		(shape input)
+		(at 55.88 60.96 180)
+		(fields_autoplaced yes)
+		(effects
+			(font
+				(size 1.27 1.27)
+			)
+			(justify right)
+		)
+		(property "Intersheetrefs" "${INTERSHEET_REFS}"
+			(at 48.2382 60.96 0)
+			(effects
+				(font
+					(size 1.27 1.27)
+				)
+				(justify right)
+				(hide yes)
+			)
+		)
+	)
 	(global_label "UART2_TX"
 		(shape input)
@@
 		)
 	)
+	(global_label "LED1"
+		(shape input)
+		(at 88.9 76.2 0)
+		(fields_autoplaced yes)
+		(effects
+			(font
+				(size 1.27 1.27)
+			)
+			(justify left)
+		)
+		(property "Intersheetrefs" "${INTERSHEET_REFS}"
+			(at 96.5418 76.2 0)
+			(effects
+				(font
+					(size 1.27 1.27)
+				)
+				(justify left)
+				(hide yes)
+			)
+		)
+	)
 	(global_label "U_OUT"
 		(shape input)
@@
 		)
 	)
+	(global_label "LED3"
+		(shape input)
+		(at 55.88 63.5 180)
+		(fields_autoplaced yes)
+		(effects
+			(font
+				(size 1.27 1.27)
+			)
+			(justify right)
+		)
+		(property "Intersheetrefs" "${INTERSHEET_REFS}"
+			(at 48.2382 63.5 0)
+			(effects
+				(font
+					(size 1.27 1.27)
+				)
+				(justify right)
+				(hide yes)
+			)
+		)
+	)
 	(global_label "W_IN"
 		(shape input)
@@
 				(hide yes)
 			)
+		)
+	)
+	(global_label "LED4"
+		(shape input)
+		(at 55.88 66.04 180)
+		(fields_autoplaced yes)
+		(effects
+			(font
+				(size 1.27 1.27)
+			)
+			(justify right)
+		)
+		(property "Intersheetrefs" "${INTERSHEET_REFS}"
+			(at 48.2382 66.04 0)
+			(effects
+				(font
+					(size 1.27 1.27)
+				)
+				(justify right)
+				(hide yes)
+			)

Commit message: 発注した
Parts:
- added C17, C18, C19, C20, C21, C22, C23, C24, C25: 10u, Capacitor_SMD:C_0805_2012Metric, symbol Device:C
- added C26: 0.1u, Capacitor_SMD:C_0603_1608Metric, symbol Device:C
- added D10: LED, LED_SMD:LED_0603_1608Metric, symbol Device:LED
- added R19: 1k, Resistor_SMD:R_0603_1608Metric, symbol Device:R
Connections:
- net +3V3: now also C26.2
- net ENCODER_OUT: now also U4.11 (PA5)
- net GND: now also C17.1, C18.1, C19.1, C20.1, C21.1, C22.1, C23.1, C24.1, C25.1, C26.1, D10.1 (K)
- net VCC: now also C1.1, C4.1, C6.1, D1.1 (K), D2.1 (K), D3.1 (K), C17.2, C18.2, C19.2, C20.2, C21.2, C22.2, C23.2, C24.2, C25.2, R19.2
- new net: D10.2 (A), R19.1
Other:
- moved on the sheet: C14, C15, C16

Commit message: V1.1発注
Parts:
- removed U5, U6: AP7375-3.3, Package_TO_SOT_SMD:SOT-23, symbol Regulator_Linear:LM1117MP-3.3
- added TP1, TP2, TP3: TestPoint, TestPoint:TestPoint_Pad_D2.0mm, symbol Connector:TestPoint
- added U5: AP7375-5, Package_TO_SOT_SMD:SOT-23, symbol Regulator_Linear:APE8865NR-15-HF-3
- added U7: AP7375-3.3, Package_TO_SOT_SMD:SOT-23, symbol Regulator_Linear:APE8865NR-15-HF-3
Connections:
- net +3V3: now also U7.2 (VO)
- net +5V: now also U5.2 (VO)
- net GND: now also U5.3 (GND), U7.3 (GND)
- net NSRT: now also J1.5 (Pin_5); no longer J1.3 (Pin_3)
- net SWCLK: now also J1.4 (Pin_4); no longer J1.5 (Pin_5)
- net SWDIO: now also J1.3 (Pin_3); no longer J1.4 (Pin_4)
- net U_OUT: now also TP3.1
- net VCC: now also U5.1 (VI), U7.1 (VI)
- net V_OUT: now also TP2.1
- net W_OUT: now also TP1.1
