File: CurcuitV2/CurcuitV2.kicad_pcb (KiCad board)
At the start: 2 copper layers, 40 x 40 mm, 42 parts, among them IC1 AS5600-ASOT, J1 Conn_01x07, J2 Conn_01x03, J3 Conn_01x02, Q1 Q_NMOS_DGS, Q2 Q_NMOS_DGS, Q3 Q_NMOS_DGS, Q4 Q_NMOS_DGS, Q5 Q_NMOS_DGS, Q6 Q_NMOS_DGS, SW1 SW_Push, SW2 SW_Push, U1 DRV8300DPWR, U2 STM32F303K8Tx, U7 AP7375-3.3

Commit message: CubeMX生成
Parts:
- added J4: Conn_01x02, Connector_JST:JST_PH_S2B-PH-K_1x02_P2.00mm_Horizontal, F.Cu at (133.6, 111.0)
- moved J1 15.2 mm to (101.5, 127.6), turned to 180 degrees
- moved U1 8.25 mm to (109.0, 119.8)
- moved U2 3.54 mm to (115.5, 108.0), turned to -90 degrees
Connections:
- U2 pad 13: unconnected-(U2-PA7-Pad13) -> INLC
- U2 pad 14: unconnected-(U2-PB0-Pad14) -> INLB
- U2 pad 15: unconnected-(U2-PB1-Pad15) -> INLA
- U2 pad 18: unconnected-(U2-PA8-Pad18) -> INHC
- U2 pad 19: unconnected-(U2-PA9-Pad19) -> INHB
- U2 pad 20: unconnected-(U2-PA10-Pad20) -> INHA

Commit message: ほぼ完成
Parts:
- added C12: 0.1u, Capacitor_SMD:C_0805_2012Metric, F.Cu at (108.0, 110.5)
- added C13: 0.1u, Capacitor_SMD:C_0805_2012Metric, F.Cu at (108.0, 108.2)
- added C14: 0.1u, Capacitor_SMD:C_0805_2012Metric, F.Cu at (108.0, 106.0)
- added C15: 0.1u, Capacitor_SMD:C_0805_2012Metric, F.Cu at (108.0, 103.8)
- added C16: 0.1u, Capacitor_SMD:C_0805_2012Metric, F.Cu at (108.0, 101.5)
- added C17: 0.1u, Capacitor_SMD:C_0805_2012Metric, F.Cu at (130.0, 102.2)
- added C18: 0.1u, Capacitor_SMD:C_0805_2012Metric, F.Cu at (129.8, 105.0)
- added C19: 0.1u, Capacitor_SMD:C_0805_2012Metric, F.Cu at (132.2, 102.2)
- added C20: 0.1u, Capacitor_SMD:C_0805_2012Metric, F.Cu at (101.5, 108.0)
- added C21: 0.1u, Capacitor_SMD:C_0805_2012Metric, F.Cu at (103.8, 108.0)
- added C22: 0.1u, Capacitor_SMD:C_0603_1608Metric, F.Cu at (110.8, 125.0)
- added C23: 0.1u, Capacitor_SMD:C_0805_2012Metric, F.Cu at (114.2, 125.2)
- added D1: 1N4148W, Diode_SMD:D_SOD-123, F.Cu at (126.5, 106.5)
- added D10: LED, LED_SMD:LED_0603_1608Metric, F.Cu at (128.0, 102.0)
- added D11: 1N4148W, Diode_SMD:D_SOD-123, F.Cu at (126.5, 123.0)
- added D12: 1N4148W, Diode_SMD:D_SOD-123, F.Cu at (118.8, 121.5)
- added D2: 1N4148W, Diode_SMD:D_SOD-123, F.Cu at (118.8, 105.0)
- added D3: 1N4148W, Diode_SMD:D_SOD-123, F.Cu at (126.5, 114.8)
- added D5: 1N4148W, Diode_SMD:D_SOD-123, F.Cu at (118.8, 113.2)
- added D6: LED, LED_SMD:LED_0603_1608Metric, F.Cu at (120.5, 138.0)
- added D7: LED, LED_SMD:LED_0603_1608Metric, F.Cu at (122.0, 138.0)
- added D8: LED, LED_SMD:LED_0603_1608Metric, F.Cu at (123.5, 138.0)
- added D9: LED, LED_SMD:LED_0603_1608Metric, F.Cu at (125.0, 138.0)
- added H1: MountingHole_Pad, MountingHole:MountingHole_3.2mm_M3_ISO14580_Pad_TopBottom, F.Cu at (137.0, 103.0)
- added H2: MountingHole_Pad, MountingHole:MountingHole_3.2mm_M3_ISO14580_Pad_TopBottom, F.Cu at (103.0, 103.0)
- added H3: MountingHole_Pad, MountingHole:MountingHole_3.2mm_M3_ISO14580_Pad_TopBottom, F.Cu at (103.0, 137.0)
- added H4: MountingHole_Pad, MountingHole:MountingHole_3.2mm_M3_ISO14580_Pad_TopBottom, F.Cu at (137.0, 137.0)
- added R15: 1k, Resistor_SMD:R_0603_1608Metric, F.Cu at (120.5, 134.8)
- added R16: 1k, Resistor_SMD:R_0603_1608Metric, F.Cu at (122.0, 134.8)
- added R17: 1k, Resistor_SMD:R_0603_1608Metric, F.Cu at (123.5, 134.8)
- added R18: 1k, Resistor_SMD:R_0603_1608Metric, F.Cu at (125.0, 134.8)
- added R19: 1k, Resistor_SMD:R_0603_1608Metric, F.Cu at (126.2, 102.0)
- added R20: 10k, Resistor_SMD:R_0603_1608Metric, F.Cu at (130.8, 129.0)
- added TP1: TestPoint, TestPoint:TestPoint_Pad_D2.5mm, B.Cu at (137.0, 116.5)
- added TP2: TestPoint, TestPoint:TestPoint_Pad_D2.5mm, B.Cu at (137.0, 120.0)
- added TP3: TestPoint, TestPoint:TestPoint_Pad_D2.5mm, B.Cu at (137.0, 123.5)
- added TP4: TestPoint, TestPoint:TestPoint_Pad_D2.5mm, B.Cu at (137.0, 108.5)
- added TP5: TestPoint, TestPoint:TestPoint_Pad_D2.5mm, B.Cu at (137.0, 112.0)
- added U3: MCP9700x-ETT, Package_TO_SOT_SMD:SOT-23, F.Cu at (118.2, 127.2)
- added Y2: CSTNE16M0V530000R0, Crystal:Resonator_SMD_Murata_CSTxExxV-3Pin_3.0x1.1mm, F.Cu at (118.2, 134.2)
- IC1: moved to B.Cu
- moved C9 58.1 mm to (116.0, 137.8), turned to 90 degrees
- moved R14 56.8 mm to (130.0, 131.5)
- moved C26 52.6 mm to (117.8, 130.8), turned to -90 degrees
- moved R13 47.1 mm to (113.2, 138.8)
- moved SW2 46.3 mm to (131.8, 136.8), turned to 90 degrees
- moved SW1 46.2 mm to (127.8, 136.8), turned to -90 degrees
- moved C10 43.5 mm to (107.0, 127.2), turned to -90 degrees
- moved IC1 43.3 mm to (120.0, 120.0), turned to 90 degrees
- moved C11 35.9 mm to (104.0, 116.2), turned to -90 degrees
- moved C8 35.5 mm to (127.2, 129.8), turned to -90 degrees
- moved U7 30.4 mm to (124.2, 130.0), turned to -90 degrees
- moved D4 29.3 mm to (124.2, 126.8), turned to 180 degrees
- moved C7 29.1 mm to (121.2, 129.8), turned to -90 degrees
- moved U2 24.8 mm to (111.5, 132.5), turned to 180 degrees
- moved J4 19.0 mm to (133.6, 130.0)
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Connections:
- C4 pad 2: GND -> GNDA
- C5 pad 2: GND -> GNDA
- C6 pad 2: GND -> GNDA
- J3 pad 1: GND -> GNDA
- J4 pad 1: unconnected-(J4-Pin_1-Pad1) -> UART2_TX
- J4 pad 2: unconnected-(J4-Pin_2-Pad2) -> UART2_RX
- Q2 pad 3: GND -> GNDA
- Q4 pad 3: GND -> GNDA
- Q6 pad 3: GND -> GNDA
- R12 pad 2: GND -> GNDA
- R3 pad 2: GND -> GNDA
- R8 pad 2: GND -> GNDA
- U1 pad 8: GND -> GNDA
- U2 pad 10: unconnected-(U2-PA4-Pad10) -> TEMP
- U2 pad 11: unconnected-(U2-PA5-Pad11) -> ENCODER_OUT
- U2 pad 2: unconnected-(U2-PF0-Pad2) -> Net-(U2-PF0)
- U2 pad 25: unconnected-(U2-PA15-Pad25) -> LED1
- U2 pad 26: unconnected-(U2-PB3-Pad26) -> LED2
- U2 pad 27: unconnected-(U2-PB4-Pad27) -> LED3
- U2 pad 28: unconnected-(U2-PB5-Pad28) -> LED4
- U2 pad 29: unconnected-(U2-PB6-Pad29) -> PC_TX
- U2 pad 3: unconnected-(U2-PF1-Pad3) -> Net-(U2-PF1)
- U2 pad 30: unconnected-(U2-PB7-Pad30) -> PC_RX
- U2 pad 6: unconnected-(U2-PA0-Pad6) -> BUTTON
- U2 pad 8: unconnected-(U2-PA2-Pad8) -> UART2_TX
- U2 pad 9: unconnected-(U2-PA3-Pad9) -> UART2_RX
Routing:
- net VCC: track 0.00 -> 82.8 mm, vias 0 -> 42
- net +3V3: track 0.00 -> 81.5 mm, vias 0 -> 3
- net GNDA: track 0.00 -> 40.4 mm, vias 0 -> 34
- net GND: track 5.63 -> 43.1 mm, vias 0 -> 33
- net NSRT: track 0.00 -> 35.6 mm, vias 0 -> 2
- net OUTA: track 0.00 -> 24.5 mm
- net UART2_RX: track 0.00 -> 22.3 mm, vias 0 -> 1
- net GHA: track 6.13 -> 28.0 mm
- net BUTTON: track 0.00 -> 21.5 mm, vias 0 -> 2
- net SWDIO: track 0.00 -> 20.2 mm
- net BSTA: track 2.26 -> 22.1 mm
- net SWCLK: track 0.00 -> 18.4 mm
- net UART2_TX: track 0.00 -> 18.1 mm, vias 0 -> 1
- net LED4: track 0.00 -> 17.7 mm, vias 0 -> 2
- net GLA: track 0.00 -> 17.5 mm, vias 0 -> 2
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- added copper zone on B.Cu, net GND
- added copper zone on F.Cu, net GND
- added copper zone on B.Cu, net GNDA
- added copper zone on F.Cu, net GNDA
- added copper zone on B.Cu, net VCC
- added copper zone on F.Cu, net VCC
Other:
- outline, holes or cut-outs redrawn
- board text added: "+"
- board text added: "-"
- board text added: "1"
- board text added: "2"
- board text added: "3"
- board text added: "3V3"
- board text added: "4"
- board text added: "CLK"
- board text added: "DIO"
- board text added: "GND"
- board text added: "NRST"
- board text added: "RST"
- board text added: "RX"
- board text added: "TX"
- board text added: "U"
- board text added: "USW"
- board text added: "V"
- board text added: "W"

Commit message: 完成
Parts:
- added NT1: NetTie_2, NetTie:NetTie-2_SMD_Pad2.0mm, B.Cu at (133.5, 125.2)
- added R21: 10k, Resistor_SMD:R_0603_1608Metric, F.Cu at (130.0, 128.2)
- added R22: 1k, Resistor_SMD:R_0603_1608Metric, F.Cu at (130.0, 126.5)
- moved R20 1.25 mm to (130.0, 130.0), turned to 180 degrees
- moved R14 0.25 mm to (130.0, 131.8)
Connections:
- U2 pad 12: unconnected-(U2-PA6-Pad12) -> VOLTAGE
Routing:
- net GND: track 43.1 -> 105.1 mm, vias 33 -> 38
- net VCC: track 82.8 -> 49.4 mm, vias 42 -> 44
- net VOLTAGE: track 0.00 -> 21.3 mm, vias 0 -> 2
- net GNDA: track 40.4 -> 55.1 mm, vias 34 -> 46
- net +3V3: track 81.5 -> 80.4 mm
- net UART2_RX: track 22.3 -> 23.0 mm
Other:
- board text added: "BLDC Driver V2.0 Designed by Bambi"

Commit message: 製造ファイル生成
Routing:
- net GNDA: track 55.1 -> 49.6 mm, vias 46 -> 47
- net GND: vias 38 -> 44
Other:
- board text removed: "NRST"
Changed lines of the file:
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@@
 		)
 	)
-	(gr_text "NRST"
+	(gr_text "RST"
 		(at 102.77 122.54 0)
 		(layer "B.SilkS")
@@
 	)
 	(via
+		(at 125.5 130.5)
+		(size 0.6)
+		(drill 0.3)
+		(layers "F.Cu" "B.Cu")
+		(free yes)
+		(net 1)
+	)
+	(via
 		(at 101.75 129)
 		(size 0.6)
@@
 	)
 	(via
+		(at 105.75 139)
+		(size 0.6)
+		(drill 0.3)
+		(layers "F.Cu" "B.Cu")
+		(free yes)
+		(net 1)
+	)
+	(via
 		(at 129.75 133.5)
 		(size 0.6)
@@
 	)
 	(via
+		(at 139 134.25)
+		(size 0.6)
+		(drill 0.3)
+		(layers "F.Cu" "B.Cu")
+		(free yes)
+		(net 1)
+	)
+	(via
 		(at 121.25 130.5)
 		(size 0.6)
@@
 	)
 	(via
+		(at 101 134.25)
+		(size 0.6)
+		(drill 0.3)
+		(layers "F.Cu" "B.Cu")
+		(free yes)
+		(net 1)
+	)
+	(via
 		(at 127.25 130.5)
 		(size 0.6)
@@
 	)
 	(via
+		(at 128.25 132.25)
+		(size 0.6)
+		(drill 0.3)
+		(layers "F.Cu" "B.Cu")
+		(free yes)
+		(net 1)
+	)
+	(via
 		(at 116 126.25)
 		(size 0.6)
@@
 	)
 	(via
-		(at 128 126.25)
+		(at 129.175 126.5)
 		(size 0.6)
 		(drill 0.3)
@@
 	)
 	(via
+		(at 125.75 138)
+		(size 0.6)
+		(drill 0.3)
+		(layers "F.Cu" "B.Cu")
+		(free yes)
+		(net 1)
+	)
+	(via
 		(at 107 126.475)
 		(size 0.6)
@@
 	)
 	(segment
-		(start 123.05 119)
-		(end 122.55 118.5)
-		(width 0.5)
-		(layer "F.Cu")
-		(net 58)
-	)
-	(segment
-		(start 123.25 118)
-		(end 123.05 118)
-		(width 0.5)
-		(layer "F.Cu")
-		(net 58)
-	)
-	(segment
 		(start 114.6375 106.575)
 		(end 114.825 106.3875)
@@
 	)
 	(segment
-		(start 123.05 109.75)
-		(end 122.55 110.25)
-		(width 0.5)
-		(layer "F.Cu")
-		(net 58)
-	)
-	(segment
 		(start 119.6 102.5)
 		(end 122.05 102.5)
@@
 	)
 	(segment
-		(start 123.25 102.5)
-		(end 123.05 102.5)
-		(width 0.5)
-		(layer "F.Cu")
-		(net 58)
-	)
-	(segment
 		(start 108.95 103.75)
 		(end 108.95 106)
@@
 	)
 	(segment
-		(start 123.25 109.75)
-		(end 123.05 109.75)
-		(width 0.5)
-		(layer "F.Cu")
-		(net 58)
-	)
-	(segment
-		(start 123.25 101.5)
-		(end 123.05 101.5)
-		(width 0.5)
-		(layer "F.Cu")
-		(net 58)
-	)
-	(segment
 		(start 118.75 103.35)
 		(end 119.6 102.5)
@@
 	)
 	(segment
-		(start 123.05 118)
-		(end 122.55 118.5)
-		(width 0.5)
-		(layer "F.Cu")
-		(net 58)
-	)
-	(segment
-		(start 123.25 110.75)
-		(end 123.05 110.75)
-		(width 0.5)
-		(layer "F.Cu")
-		(net 58)
-	)
-	(segment
 		(start 122.05 102.5)
 		(end 122.55 102)
@@
 	)
 	(segment
-		(start 123.05 102.5)
-		(end 122.55 102)
-		(width 0.5)
-		(layer "F.Cu")
-		(net 58)
-	)
-	(segment
 		(start 114.825 124.875)
 		(end 114.825 122.8875)
@@
 	)
 	(segment
-		(start 123.05 110.75)
-		(end 122.55 110.25)
-		(width 0.5)
-		(layer "F.Cu")
-		(net 58)
-	)
-	(segment
 		(start 122.05 110.75)
 		(end 122.55 110.25)
@@
 	)
 	(segment
-		(start 123.25 119)
-		(end 123.05 119)
-		(width 0.5)
-		(layer "F.Cu")
-		(net 58)
-	)
-	(segment
 		(start 132.25 101.3)
 		(end 133.45 101.3)
@@
 	)
 	(segment
-		(start 123.05 101.5)
-		(end 122.55 102)
-		(width 0.5)
-		(layer "F.Cu")
-		(net 58)
-	)
-	(segment
 		(start 118.75 119.85)
 		(end 119.6 119)
@@
 	)
 	(via
-		(at 123.25 119)
+		(at 110 118.5)
 		(size 0.6)
 		(drill 0.3)
@@
 	)
 	(via
-		(at 110 118.5)
+		(at 112.75 108.25)
 		(size 0.6)
 		(drill 0.3)
@@
 	)
 	(via
-		(at 112.75 108.25)
+		(at 117.75 119)
 		(size 0.6)
 		(drill 0.3)
@@
 	)
 	(via
-		(at 117.75 119)
+		(at 105.5 118.5)
 		(size 0.6)
 		(drill 0.3)
@@
 	)
 	(via
-		(at 105.5 118.5)
+		(at 118.75 103.5)
 		(size 0.6)
 		(drill 0.3)
@@
 	)
 	(via
-		(at 132 116)
+		(at 132.25 116)
 		(size 0.6)
 		(drill 0.3)
@@
 	)
 	(via
-		(at 123.25 102.5)
+		(at 122.75 118)
 		(size 0.6)
 		(drill 0.3)
@@
 	)
 	(via
-		(at 123.25 118)
+		(at 135.25 124)
 		(size 0.6)
 		(drill 0.3)
@@
 	)
 	(via
-		(at 123.25 109.75)
+		(at 139 105.75)
 		(size 0.6)
 		(drill 0.3)
@@
 	)
 	(via
-		(at 135.25 124)
+		(at 101 110)
 		(size 0.6)
 		(drill 0.3)
@@
 	)
 	(via
-		(at 101 110)
+		(at 130.25 110.461991)
 		(size 0.6)
 		(drill 0.3)
@@
 	)
 	(via
-		(at 130.25 110.461991)
+		(at 122.75 109.75)
 		(size 0.6)
 		(drill 0.3)
 		(layers "F.Cu" "B.Cu")
-		(free yes)
 		(net 58)
 	)
@@
 	)
 	(via
-		(at 139 114.5)
+		(at 118.75 111.75)
 		(size 0.6)
 		(drill 0.3)
@@
 	)
 	(via
-		(at 123.25 101.5)
+		(at 139 114.5)
 		(size 0.6)
 		(drill 0.3)
@@
 	)
 	(via
-		(at 123.25 110.75)
+		(at 118.75 119.5)
 		(size 0.6)
 		(drill 0.3)
@@
 	)
 	(via
+		(at 122.75 102.5)
+		(size 0.6)
+		(drill 0.3)
+		(layers "F.Cu" "B.Cu")
+		(free yes)
+		(net 58)
+	)
+	(via
 		(at 105.5 121.5)
 		(size 0.6)
@@
 			(pts
 				(xy 116.25 109.5) (xy 116.25 111) (xy 115.5 111.75) (xy 115.5 114.75) (xy 118 117.25) (xy 125 117.25)
-				(xy 128.5 120.75) (xy 130.5 120.75) (xy 130.5 119.25) (xy 130.25 119.25) (xy 126.75 115.75) (xy 123.25 115.75)
-				(xy 122.75 115.25) (xy 122.75 114) (xy 119.75 114) (xy 117.25 111.5) (xy 117.25 109.5)
+				(xy 128.5 120.75) (xy 130.5 120.75) (xy 130.5 119.25) (xy 127 115.75) (xy 123.25 115.75) (xy 122.75 115.25)
+				(xy 122.75 114) (xy 119.75 114) (xy 117.25 111.5) (xy 117.25 109.5)
 			)
 		)
@@
 			(pts
 				(xy 116.25 101.25) (xy 116.25 102.75) (xy 115.5 103.5) (xy 115.5 106.5) (xy 118 109) (xy 125 109)
-				(xy 127.5 111.5) (xy 127.5 115.75) (xy 130 118.25) (xy 131.25 118.25) (xy 131.25 114.5) (xy 129.25 112.5)
+				(xy 127.5 111.5) (xy 127.5 115.75) (xy 130 118.25) (xy 131.5 118.25) (xy 131.5 114.75) (xy 129.25 112.5)
 				(xy 129.25 110.03125) (xy 127 107.5) (xy 123.25 107.5) (xy 122.75 107) (xy 122.75 105.75) (xy 119.75 105.75)
 				(xy 117.25 103.25) (xy 117.25 101.25)
