File: CurcuitV3/CurcuitV3.kicad_pcb (KiCad board)
At the start: 2 copper layers, 40 x 40 mm, 92 parts, among them IC1 AS5600-ASOT, J1 Conn_01x07, J2 Conn_01x03, J3 Conn_01x02, J4 Conn_01x02, Q1 Q_NMOS_DGS, Q2 Q_NMOS_DGS, Q3 Q_NMOS_DGS, Q4 Q_NMOS_DGS, Q5 Q_NMOS_DGS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

Commit message: 電流センス部品の追加
Parts:
- added R26: 10m, Resistor_SMD:R_1206_3216Metric, F.Cu at (151.0, 113.8)
- added R27: 10m, Resistor_SMD:R_1206_3216Metric, F.Cu at (151.0, 116.8)
- added U5: INA180A2, Package_TO_SOT_SMD:SOT-23-5, F.Cu at (145.6, 114.2)
- added U6: INA180A2, Package_TO_SOT_SMD:SOT-23-5, F.Cu at (145.6, 118.8)
Connections:
- C1 pad 1: OUTA -> Net-(D1-A)
- C2 pad 1: OUTB -> Net-(D3-A)
- D1 pad 2: OUTA -> Net-(D1-A)
- D2 pad 1: OUTA -> Net-(D1-A)
- D3 pad 2: OUTB -> Net-(D3-A)
- D5 pad 1: OUTB -> Net-(D3-A)
- Q1 pad 3: OUTA -> Net-(D1-A)
- Q2 pad 1: OUTA -> Net-(D1-A)
- Q3 pad 3: OUTB -> Net-(D3-A)
- Q4 pad 1: OUTB -> Net-(D3-A)
- R4 pad 2: OUTA -> Net-(D1-A)
- R7 pad 2: OUTB -> Net-(D3-A)
