File: CurcuitV3/CurcuitV3.kicad_pcb (KiCad board)
At the start: 2 copper layers, 40 x 40 mm, 97 parts, among them IC1 AS5600-ASOT, J1 Conn_01x02, J2 Conn_01x03, J3 Conn_01x07, J4 Conn_01x02, Q1 Q_NMOS_DGS, Q2 Q_NMOS_DGS, Q3 Q_NMOS_DGS, Q4 Q_NMOS_DGS, Q5 Q_NMOS_DGS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

Commit message: ほぼ完成
Parts:
- removed C12, C20, C21: 10u, Capacitor_SMD:C_0805_2012Metric
- C4: value 10u -> 100u; footprint Capacitor_SMD:C_0805_2012Metric -> Capacitor_THT:CP_Radial_D6.3mm_P2.50mm
- C5: footprint Capacitor_SMD:C_0805_2012Metric -> Capacitor_SMD:C_0603_1608Metric
- C7: value 0.1u -> 100u; footprint Capacitor_SMD:C_0603_1608Metric -> Capacitor_THT:CP_Radial_D6.3mm_P2.50mm
- C8: value 10u -> 0.1u; footprint Capacitor_SMD:C_0805_2012Metric -> Capacitor_SMD:C_0603_1608Metric
- J2: footprint Connector_JST:JST_XH_S3B-XH-A_1x03_P2.50mm_Horizontal -> Connector_Molex:Molex_SPOX_5268-03A_1x03_P2.50mm_Horizontal
- J4: footprint Connector_JST:JST_XH_S2B-XH-A_1x02_P2.50mm_Horizontal -> Connector_Molex:Molex_SPOX_5268-02A_1x02_P2.50mm_Horizontal
- R14, R21: value 10m -> 10; footprint Resistor_SMD:R_1206_3216Metric -> Resistor_SMD:R_0603_1608Metric
- R15, R22: value 10 -> 10k
- R16, R24: value 10k -> 10m; footprint Resistor_SMD:R_0603_1608Metric -> Resistor_SMD:R_1206_3216Metric
- U5: footprint Package_TO_SOT_SMD:SOT-363_SC-70-6 -> Package_TO_SOT_SMD:Texas_R-PDSO-G6
- moved R15 99.9 mm to (119.0, 114.0)
- moved C8 98.8 mm to (111.5, 125.8), turned to 180 degrees
- moved Q4 98.3 mm to (121.8, 113.5)
- moved D8 98.2 mm to (122.8, 116.8), turned to 180 degrees
- moved D7 97.1 mm to (130.2, 116.5)
- moved Q3 96.4 mm to (127.2, 113.5)
- moved C9 96.3 mm to (127.2, 110.2)
- moved R12 96.3 mm to (124.5, 110.8)
- moved R13 96.3 mm to (124.5, 114.0)
- moved R16 95.8 mm to (115.5, 115.0), turned to 180 degrees
- moved C10 93.8 mm to (132.5, 102.0)
- moved C11 87.2 mm to (130.2, 102.0)
- moved R14 86.7 mm to (119.0, 110.8), turned to -90 degrees
- moved R23 81.7 mm to (130.0, 127.8)
- moved C24 79.9 mm to (130.0, 129.5)
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Connections:
- C10 pad 1: GNDA -> GNDPWR
- C11 pad 1: GNDA -> GNDPWR
- C13 pad 1: GNDA -> GNDPWR
- C14 pad 1: GNDA -> GNDPWR
- C15 pad 1: GNDA -> GNDPWR
- C2 pad 2: GNDA -> GNDPWR
- C22 pad 1: Net-(D10-K) -> OUTC
- C23 pad 2: GNDA -> GNDPWR
- C4 pad 1: GNDA -> VCC
- C4 pad 2: VCC -> GNDPWR
- C5 pad 1: GNDA -> GNDPWR
- C6 pad 1: GNDA -> OUTB
- C6 pad 2: VCC -> BSTB
- C7 pad 1: GNDA -> VCC
- C7 pad 2: VCC -> GNDPWR
- C8 pad 1: Net-(D7-A) -> GNDPWR
- C8 pad 2: BSTB -> VCC
- C9 pad 2: GNDA -> GNDPWR
- D10 pad 1: Net-(D10-K) -> OUTC
- D10 pad 2: GNDA -> Net-(D10-A)
- D12 pad 1: GNDA -> GNDPWR
- D6 pad 2: GNDA -> GNDPWR
- D7 pad 2: Net-(D7-A) -> OUTB
- D8 pad 1: Net-(D7-A) -> OUTB
- D8 pad 2: GNDA -> Net-(D8-A)
- D9 pad 2: Net-(D10-K) -> OUTC
- J4 pad 1: GNDA -> GNDPWR
- NT1 pad 2: GNDA -> GNDPWR
- Q2 pad 3: GNDA -> GNDPWR
- Q3 pad 3: Net-(D7-A) -> OUTB
- Q4 pad 1: Net-(D7-A) -> OUTB
- Q4 pad 3: GNDA -> Net-(D8-A)
- Q5 pad 3: Net-(D10-K) -> OUTC
- Q6 pad 1: Net-(D10-K) -> OUTC
- Q6 pad 3: GNDA -> Net-(D10-A)
- R10 pad 2: GNDA -> GNDPWR
- R13 pad 2: Net-(D7-A) -> OUTB
- R14 pad 1: Net-(D7-A) -> GLB
- R14 pad 2: OUTB -> Net-(Q4-G)
- R15 pad 1: GLB -> Net-(Q4-G)
- R15 pad 2: Net-(Q4-G) -> Net-(D8-A)
- R16 pad 1: Net-(Q4-G) -> Net-(D8-A)
- R16 pad 2: GNDA -> GNDPWR
- R20 pad 2: Net-(D10-K) -> OUTC
- R21 pad 1: Net-(D10-K) -> GLC
- R21 pad 2: OUTC -> Net-(Q6-G)
- R22 pad 1: GLC -> Net-(Q6-G)
- R22 pad 2: Net-(Q6-G) -> Net-(D10-A)
- R23 pad 1: Net-(Q6-G) -> VOLTAGE
- R23 pad 2: GNDA -> VCC
- R24 pad 1: VOLTAGE -> Net-(D10-A)
- R24 pad 2: VCC -> GNDPWR
- TP4 pad 1: GNDA -> GNDPWR
- U1 pad 8: GNDA -> GNDPWR
- U2 pad 21: BUTTON -> USB
- U2 pad 22: USB -> BUTTON
- U4 pad 3: Net-(D7-A) -> Net-(D8-A)
- U4 pad 4: OUTB -> GNDPWR
- U6 pad 1: SENSEB -> SENSEC
- U6 pad 3: Net-(D10-K) -> Net-(D10-A)
- U6 pad 4: OUTC -> GNDPWR
Routing:
- net +3V3: track 0.00 -> 114.2 mm, vias 0 -> 13
- net NSRT: track 0.00 -> 45.3 mm, vias 0 -> 6
- net BUTTON: track 0.00 -> 36.5 mm, vias 0 -> 3
- net GND: track 0.00 -> 30.5 mm, vias 0 -> 57
- net VCC: track 0.00 -> 28.1 mm, vias 0 -> 88
- net GHA: track 0.00 -> 27.4 mm, vias 0 -> 2
- net UART2_RX: track 0.00 -> 27.0 mm, vias 0 -> 1
- net VOLTAGE: track 0.00 -> 25.4 mm, vias 0 -> 2
- net OUTA: track 0.00 -> 25.3 mm
- net USB: track 0.00 -> 25.1 mm
- net BSTA: track 0.00 -> 24.5 mm
- net OUTB: track 0.00 -> 23.7 mm
- net SENSEB: track 0.00 -> 21.1 mm, vias 0 -> 2
- net GHB: track 0.00 -> 21.0 mm, vias 0 -> 2
- net SWDIO: track 0.00 -> 20.2 mm
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- added copper zone on B.Cu, net GND
- added copper zone on F.Cu, net GND
- added copper zone on B.Cu, net GNDPWR
- added copper zone on F.Cu, net GNDPWR
- added copper zone on F.Cu, net Net-(D10-A)
- added copper zone on F.Cu, net Net-(D8-A)
- added copper zone on F.Cu, net Net-(Q1-G)
- added copper zone on F.Cu, net Net-(Q2-G)
- added copper zone on F.Cu, net Net-(Q3-G)
- added copper zone on F.Cu, net Net-(Q4-G)
- added copper zone on F.Cu, net Net-(Q5-G)
- added copper zone on F.Cu, net Net-(Q6-G)
- added copper zone on F.Cu, net OUTA
- added copper zone on F.Cu, net OUTB
- added copper zone on F.Cu, net OUTC
- added copper zone on B.Cu, net VCC
- added copper zone on F.Cu, net VCC

Commit message: シルク書いた
Parts:
- added C12: 10u, Capacitor_SMD:C_0805_2012Metric, F.Cu at (137.6, 132.8)
Routing:
- net GND: track 30.5 -> 1.00 mm, vias 57 -> 82
- net +3V3: track 114.2 -> 118.6 mm
- net VCC: vias 88 -> 93
- net GNDPWR: vias 67 -> 99
Other:
- board text added: "+"
- board text added: "-"
- board text added: "3V3"
- board text added: "BLDC Driver V3.0 Designed by Bambi"
- board text added: "CLK"
- board text added: "DIO"
- board text added: "DRV8300"
- board text added: "GND"
- board text added: "MOTOR"
- board text added: "POWER"
- board text added: "RST"
- board text added: "RX"
- board text added: "STM32 F303K8"
- board text added: "TX"
- board text added: "U"
- board text added: "UART"
- board text added: "V"
- board text added: "VCC"
- board text added: "W"

Commit message: 製造ファイル生成
Routing:
- net GND: vias 82 -> 86
Changed lines of the file:
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@@
+	)
+	(via
+		(at 124.25 131.25)
+		(size 0.6)
+		(drill 0.3)
+		(layers "F.Cu" "B.Cu")
+		(free yes)
+		(net 1)
 	)
 	(via
@@
 	)
 	(via
+		(at 118.911708 127.1)
+		(size 0.6)
+		(drill 0.3)
+		(layers "F.Cu" "B.Cu")
+		(free yes)
+		(net 1)
+	)
+	(via
 		(at 120.690686 126.559314)
 		(size 0.6)
@@
 	)
 	(via
+		(at 121.290686 127.159314)
+		(size 0.6)
+		(drill 0.3)
+		(layers "F.Cu" "B.Cu")
+		(free yes)
+		(net 1)
+	)
+	(via
 		(at 105.210769 139.45)
 		(size 0.6)
@@
 		(size 0.6)
 		(drill 0.3)
+		(layers "F.Cu" "B.Cu")
+		(free yes)
+		(net 1)
+	)
+	(via
+		(at 132.196814 132.528186)
+		(size 0.6)
+		(drill 0.3)
