File: CurcuitV3/CurcuitV3.kicad_pcb (KiCad board)
At the start: 2 copper layers, 40 x 40 mm, 95 parts, among them IC1 AS5600-ASOT, J1 Conn_01x02, J2 Conn_01x03, J3 Conn_01x07, J4 Conn_01x02, Q1 Q_NMOS_DGS, Q2 Q_NMOS_DGS, Q3 Q_NMOS_DGS, Q4 Q_NMOS_DGS, Q5 Q_NMOS_DGS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

Commit message: V3の修正と製造ファイル生成
Parts:
- moved NT1 1.25 mm to (139.5, 125.5)
- moved C14 0.78 mm to (108.8, 104.0)
- moved C15 0.78 mm to (108.8, 102.0)
- moved C10 0.25 mm to (132.2, 102.0)
Connections:
- U4 pad 2: GND -> GNDPWR
- U6 pad 2: GND -> GNDPWR
Routing:
- net VCC: track 28.1 -> 25.2 mm, vias 93 -> 96
- net +3V3: track 118.6 -> 121.0 mm
- net SENSEB: track 21.1 -> 21.7 mm
- net SENSEC: track 9.45 -> 9.96 mm
- net GNDPWR: vias 99 -> 106
- net GND: vias 86 -> 89
