File: CurcuitV3/_autosave-CurcuitV3.kicad_pcb (KiCad board)
At the start: 2 copper layers, 40 x 40 mm, 97 parts, among them IC1 AS5600-ASOT, J1 Conn_01x02, J2 Conn_01x03, J3 Conn_01x07, J4 Conn_01x02, Q1 Q_NMOS_DGS, Q2 Q_NMOS_DGS, Q3 Q_NMOS_DGS, Q4 Q_NMOS_DGS, Q5 Q_NMOS_DGS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

Commit message: 回路ほぼ完成
Parts:
- U4, U6: moved to B.Cu
- moved U4 54.1 mm to (43.8, 68.2), turned to 0 degrees
- moved D10 24.0 mm to (103.5, 67.0)
- moved U6 23.8 mm to (107.8, 70.2)
- moved R19 19.6 mm to (105.5, 64.2)
- moved R22 18.2 mm to (97.8, 64.2), turned to -90 degrees
- moved R23 13.4 mm to (97.8, 67.5), turned to -90 degrees
- moved R21 13.3 mm to (107.8, 70.5), turned to 0 degrees
- moved U5 11.2 mm to (87.9, 112.0)
- moved R20 2.51 mm to (105.5, 67.5), turned to -90 degrees
- moved R14 0.25 mm to (43.5, 68.5)
