File: CurcuitV4/CurcuitV4.kicad_sch (KiCad schematic)
At the start: 95 parts, among them IC1 AS5600-ASOT, J1 Conn_01x02, J2 Conn_01x03, J3 Conn_01x07, J4 Conn_01x02, Q1 Q_NMOS_DGS, Q2 Q_NMOS_DGS, Q3 Q_NMOS_DGS, Q4 Q_NMOS_DGS, Q5 Q_NMOS_DGS, Q6 Q_NMOS_DGS, SW1 SW_Push, SW2 SW_Push, U1 DRV8300DPWR, U2 STM32F303K8Tx, U3 MCP9700x-ETT, U4 INA181, U6 INA181, U7 AP7375-3.3, Y1 CSTNE16M0V530000R0

Commit message: TVSダイオードの追加とGNDビア増やした
Parts:
- added C14: 1u, Capacitor_SMD:C_0603_1608Metric, symbol Device:C
- added D14: SMAJ13A, Diode_SMD:D_SMA, symbol Diode:SMAJ13A
Connections:
- net +3V3: now also C14.2
- net GND: now also C14.1
- net GNDPWR: now also D14.2 (A2)
- net VCC: now also D14.1 (A1)
